File: UartTempSens.kicad_pcb (KiCad board)
At the start: 2 copper layers, 60.5 x 25 mm, 35 parts, among them J1 Conn_01x02, J2 Conn_01x02, J3 Conn_01x02, J4 USB_B_Micro, J5 Conn_01x05, SW1 SW_Push, U1 MIC5504-3.3YM5, U2 STM32G0B1KCTx, U3 OLED Display, U4 USBLC6-2SC6

Commit message: Fix library path
Parts:
- U3: footprint SCOLIB:SMIH-05VDC-SL-C, OLED DISPLAY, 128x64 -> personal-lib:SMIH-05VDC-SL-C,OLED_DISPLAY,128x64
