File: UartTempSens.kicad_sch (KiCad schematic)
At the start: 35 parts, among them J1 Conn_01x02, J2 Conn_01x02, J3 Conn_01x02, J4 USB_B_Micro, J5 Conn_01x05, SW1 SW_Push, U1 MIC5504-3.3YM5, U2 STM32G0B1KCTx, U3 OLED Display, U4 USBLC6-2SC6

Commit message: Fix library path
Parts:
- removed U3: OLED Display, SCOLIB:SMIH-05VDC-SL-C, OLED DISPLAY, 128x64, symbol Personal_lib:1,3''_SPI_OLED_Display,_64x128
- added U3: OLED Display, personal-lib:SMIH-05VDC-SL-C,OLED_DISPLAY,128x64, symbol personal-lib:1,3''_SPI_OLED_Display,_64x128
Connections:
- net +3V3: now also U3.2 (VCC)
- net DISP_CS: now also U3.7 (CS)
- net DISP_DC: now also U3.6 (DC)
- net DISP_RST: now also U3.5 (nRST)
- net GND: now also U3.1 (GND), U3.8 (MH1), U3.9 (MH2)
- net SPI1_MOSI: now also U3.4 (MOSI)
- net SPI1_SCK: now also U3.3 (SCLK)
